File: flight/targets/sparky2/hw/kicad/Sparky2.sch (KiCad schematic (older format))
At the start: 80 parts, among them Q1_2 Dual N MOSFET, Q2 Dual N MOSFET, U1 STM32F405RGT6, U2 LP2992-3.3, U3 CAN Transceiver, U6 XOR, U7 Pressure Sensor, U9 Flash 16Mbits

Commit message: Sparky2: update kicad schematic following fixes in converter
This fixes the power port symbols.
Connections:
- net labels added: +VCC, +VCC_UNREG
- net labels removed: +1.2V
